File: pcbDesignForAutonomousDrivingProject.kicad_pcb (KiCad board)
At the start: 2 copper layers, 200 x 239 mm, 26 parts, among them J1 Wheel Encoder, J2 Jack-DC, U1 can, U10 can, U11 GPSModule, U12 SJ2Board, U13 can, U14 SJ2Board, U15 can, U16 DAC, U17 motorTransceiver, U18 can, U19 OLED, U2 SJ2Board, U20 ESP8266, U21 SJ2Board, U22 12vto5v, U3 SJ2Board, U4 Compass, U5 ultrasonic, U6 ultrasonic, U7 ultrasonic, U8 ultrasonic, U9 ultrasonic

Commit message: Commit Made on - April 25th 2021 @ 03:14:31 PM
Parts:
- U14: moved to F.Cu
- moved U14 296.7 mm to (48.0, -87.0), turned to 90 degrees
- moved U12 235.4 mm to (163.0, -141.0)
- moved U3 224.1 mm to (157.0, -62.0), turned to 90 degrees
- moved U2 164.0 mm to (228.0, -62.0)
- moved U21 57.7 mm to (234.0, -141.0), turned to 270 degrees
- moved U9 44.0 mm to (47.0, -347.0)
- moved U6 26.0 mm to (63.0, -188.7)
Other:
- board size 200 x 239 mm -> 140 x 140 mm

Commit message: Commit Made on - April 25th 2021 @ 11:22:35 PM
Parts:
- added J3: CanHL, Connector_PinHeader_2.54mm:PinHeader_1x02_P2.54mm_Vertical, F.Cu at (195.0, -127.0)
- C1: footprint Capacitor_THT:CP_Radial_D8.0mm_P3.80mm -> Capacitor_THT:CP_Radial_D5.0mm_P2.50mm
- U14: moved to B.Cu
- U21: moved to F.Cu
- moved U16 628.1 mm to (245.0, -159.0)
- moved U19 623.5 mm to (194.0, -149.0)
- moved J1 609.3 mm to (259.0, -93.0), turned to 180 degrees
- moved C1 599.3 mm to (237.0, -75.0), turned to 180 degrees
- moved U11 589.9 mm to (157.0, -150.0), turned to 90 degrees
- moved R1 588.9 mm to (237.0, -82.0), turned to 180 degrees
- moved U17 568.9 mm to (259.0, -111.0), turned to 180 degrees
- moved U20 553.0 mm to (244.0, -142.0)
- moved U4 532.0 mm to (220.0, -150.0), turned to 90 degrees
- moved U8 492.4 mm to (196.0, -39.0), turned to 90 degrees
- moved U15 463.6 mm to (146.0, -126.0), turned to 180 degrees
- moved U10 440.0 mm to (176.0, -125.0)
- moved U18 420.7 mm to (245.0, -125.0)
- moved U13 395.2 mm to (215.0, -126.0), turned to 180 degrees
- moved U5 382.3 mm to (196.0, -169.0), turned to 180 degrees
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Connections:
- J1 pad 1: 3.3v -> 3.3vDACNode
- U1 pad 3: 3.3v -> 3.3vUlSo
- U10 pad 3: 3.3v -> 3.3vGPSNode
- U11 pad 0: 3.3v -> 3.3vGPSNode
- U12 pad 4: Net-(U12-Pad4) -> 3.3vDACNode
- U13 pad 3: 3.3v -> 3.3vDriverNode
- U14 pad 4: Net-(U14-Pad4) -> 3.3vDriverNode
- U15 pad 3: 3.3v -> 3.3vDACNode
- U17 pad 1: 5v -> 3.3vDACNode
- U18 pad 3: 3.3v -> 3.3vbridgeNode
- U2 pad 4: Net-(U2-Pad4) -> 3.3vUlSo
- U20 pad 5: 3.3v -> 3.3vbridgeNode
- U20 pad 7: 3.3v -> 3.3vbridgeNode
- U21 pad 4: Net-(U21-Pad4) -> 3.3vbridgeNode
- U3 pad 4: Net-(U3-Pad4) -> 3.3vGPSNode
- U4 pad 7: 3.3v -> 3.3vGPSNode
- U5 pad 1: 3.3v -> 3.3vUlSo
- U6 pad 1: 3.3v -> 3.3vUlSo
- U7 pad 1: 3.3v -> 3.3vUlSo
- U8 pad 1: 3.3v -> 3.3vUlSo
- U9 pad 1: 3.3v -> 3.3vUlSo
Other:
- net class Default: trace_width 0.25 -> 0.4
- net class Power added: clearance 0.3, trace_width 0.6, via_dia 0.8, via_drill 0.4
- board text added: "Bridge Node"
- board text added: "CanH"
- board text added: "CanL"
- board text added: "Driver Node"
- board text added: "GPS Node"
- board text added: "Ultrasonic Node"
- board text added: "motorTxRx Node"
