File: pcbDesignForAutonomousDrivingProject.kicad_pcb (KiCad board)
At the start: 2 copper layers, 140 x 140 mm, 27 parts, among them J1 Wheel Encoder, J2 Jack-DC, J3 CanHL, U1 can, U10 can, U11 GPSModule, U12 SJ2Board, U13 can, U14 SJ2Board, U15 can, U16 DAC, U17 motorTransceiver, U18 can, U19 OLED, U2 SJ2Board, U20 ESP8266, U21 SJ2Board, U22 12vto5v, U3 SJ2Board, U4 Compass, U5 ultrasonic, U6 ultrasonic, U7 ultrasonic, U8 ultrasonic, U9 ultrasonic

Commit message: Commit Made on - April 27th 2021 @ 10:09:59 AM
Other:
- outline, holes or cut-outs redrawn
- net class Power: trace_width 0.6 -> 0.8; via_dia 0.8 -> 1; via_drill 0.4 -> 0.5

Commit message: Commit Made on - April 27th 2021 @ 01:52:08 PM
Other:
- board text added: "12V input <-"
- board text added: "12v to 5v Converter"
- board text added: "CAN"
- board text added: "Compass"
- board text added: "DAC"
- board text added: "ESP8266"
- board text added: "GPS Module"
- board text added: "Oled"
- board text added: "Ultrasonic"

Commit message: Commit Made on - April 28th 2021 @ 11:39:06 PM
Parts:
- removed C1: C, Capacitor_THT:CP_Radial_D5.0mm_P2.50mm
- removed J1: Wheel Encoder, myFootprint:WheelEncoder
- removed J2: Jack-DC, Connector_BarrelJack:BarrelJack_CUI_PJ-102AH_Horizontal
- removed J3: CanHL, Connector_PinHeader_2.54mm:PinHeader_1x02_P2.54mm_Vertical
- removed R1: R, Resistor_THT:R_Axial_DIN0309_L9.0mm_D3.2mm_P2.54mm_Vertical
- removed U1, U10, U13, U15, U18: can, myFootprint:can
- removed U11: GPSModule, myFootprint:GPS
- removed U12, U14, U2, U21, U3: SJ2Board, myFootprint:sj2Board
- removed U16: DAC, myFootprint:DAC
- removed U17: motorTransceiver, myFootprint:motorTransceiver
- removed U19: OLED, myFootprint:Oled
- removed U20: ESP8266, myFootprint:ESP8266
- removed U22: 12vto5v, myFootprint:12vto5v
- removed U4: Compass, myFootprint:compass
- removed U5, U6, U7, U8, U9: ultrasonic, myFootprint:ultrasonic
Other:
- board text removed: "12V input <-"

Commit message: Commit Made on - April 29th 2021 @ :36:51
Parts:
- added J1: Wheel Encoder, myFootprint:WheelEncoder, F.Cu at (44.5, 156.2)
- added J2: Jack-DC, myFootprint:BarrelJack_Horizontal, F.Cu at (152.4, 145.4)
- added J3: CanHL, Connector_PinHeader_2.54mm:PinHeader_1x02_P2.54mm_Vertical, F.Cu at (90.8, 91.4)
- added J4: Input, Connector_PinHeader_2.54mm:PinHeader_1x02_P2.54mm_Vertical, F.Cu at (156.2, 125.7)
- added U1: can, myFootprint:can, F.Cu at (110.5, 69.2)
- added U10: can, myFootprint:can, F.Cu at (71.1, 69.2)
- added U11: GPSModule, myFootprint:GPS, F.Cu at (38.1, 56.5)
- added U12: SJ2Board, myFootprint:sj2Board, B.Cu at (52.1, 134.0)
- added U13: can, myFootprint:can, F.Cu at (110.5, 116.2)
- added U14: SJ2Board, myFootprint:sj2Board, B.Cu at (122.6, 134.0)
- added U15: can, myFootprint:can, F.Cu at (71.1, 116.2)
- added U16: DAC, myFootprint:DAC, F.Cu at (34.3, 128.9)
- added U17: motorTransceiver, myFootprint:motorTransceiver, F.Cu at (64.1, 155.6)
- added U19: OLED, myFootprint:Oled, F.Cu at (120.7, 34.9)
- added U2: SJ2Board, myFootprint:sj2Board, B.Cu at (128.9, 52.7)
- added U20: ESP8266, myFootprint:ESP8266, F.Cu at (146.1, 47.0)
- added U22: 12vto5v, myFootprint:12vto5v, F.Cu at (108.6, 145.4)
- added U3: SJ2Board, myFootprint:sj2Board, B.Cu at (58.4, 52.7)
- added U4: Compass, myFootprint:compass, F.Cu at (90.2, 44.5)
- added U5: ultrasonic, myFootprint:ultrasonic, F.Cu at (91.4, 29.8)
- added U6: ultrasonic, myFootprint:ultrasonic, F.Cu at (29.8, 160.0)
- added U7: ultrasonic, myFootprint:ultrasonic, F.Cu at (152.4, 160.0)
- added U8: ultrasonic, myFootprint:ultrasonic, F.Cu at (152.4, 29.8)
- added U9: ultrasonic, myFootprint:ultrasonic, F.Cu at (29.2, 29.8)
Other:
- board size 140 x 140 mm -> 145 x 145 mm
- net class Power: trace_width 0.8 -> 1; via_dia 1 -> 1.4; via_drill 0.5 -> 0.8
- board text added: "12v"
- board text added: "GND"
- board text removed: "Bridge Node"

Commit message: Commit Made on - April 29th 2021 @ :52:21
Parts:
- moved J1 328.8 mm to (259.0, -93.0)
- moved J2 243.9 mm to (248.0, -79.0), turned to 90 degrees
Changed lines of the file:
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@@
   )
   (module myFootprint:WheelEncoder (layer F.Cu)
-    (at 44.45 156.21 180)
+    (at 259 -93 180)
     (fp_text reference J1 (at -6.35 -1.905 270) (layer F.SilkS)
       (effects (font (size 1 1) (thickness 0.15)))
@@
   )
   (module myFootprint:BarrelJack_Horizontal (layer F.Cu)
-    (at 152.4 145.415 180)
+    (at 248 -79 90)
     (descr "DC Barrel Jack")
     (tags "Power Jack")
-    (fp_text reference J2 (at -8.45 5.75) (layer F.SilkS)
+    (fp_text reference J2 (at -8.45 5.75 -90) (layer F.SilkS)
       (effects (font (size 1 1) (thickness 0.15)))
     )
-    (fp_text value Jack-DC (at -6.2 -5.5) (layer F.Fab)
+    (fp_text value Jack-DC (at -6.2 -5.5 -90) (layer F.Fab)
       (effects (font (size 1 1) (thickness 0.15)))
     )
@@
     (fp_line (start 0.8 4.5) (end 0.8 -3.75) (layer F.Fab) (width 0.1))
     (fp_line (start 0 -4.5) (end -13.7 -4.5) (layer F.Fab) (width 0.1))
-    (fp_text user %R (at -3 -2.95) (layer F.Fab)
+    (fp_text user %R (at -3 -2.95 -90) (layer F.Fab)
       (effects (font (size 1 1) (thickness 0.15)))
     )
-    (pad 1 thru_hole rect (at 0 0 180) (size 3.5 3.5) (drill oval 1 3) (layers *.Cu *.Mask)
+    (pad 1 thru_hole rect (at 0 0 90) (size 3.5 3.5) (drill oval 1 3) (layers *.Cu *.Mask)
       (net 3 "Net-(J2-Pad1)"))
-    (pad 2 thru_hole roundrect (at -6 0 180) (size 3 3.5) (drill oval 1 3) (layers *.Cu *.Mask) (roundrect_rratio 0.25)
+    (pad 2 thru_hole roundrect (at -6 0 90) (size 3 3.5) (drill oval 1 3) (layers *.Cu *.Mask) (roundrect_rratio 0.25)
       (net 4 "Net-(J2-Pad2)"))
-    (pad 2 thru_hole roundrect (at -3 4.7 180) (size 3.5 3.5) (drill oval 3 1) (layers *.Cu *.Mask) (roundrect_rratio 0.25)
+    (pad 2 thru_hole roundrect (at -3 4.7 90) (size 3.5 3.5) (drill oval 3 1) (layers *.Cu *.Mask) (roundrect_rratio 0.25)
       (net 4 "Net-(J2-Pad2)"))
     (model ${KISYS3DMOD}/Connector_BarrelJack.3dshapes/BarrelJack_Horizontal.wrl

Commit message: Commit Made on - April 29th 2021 @ :53:10
Parts:
- moved J1 328.5 mm to (45.2, 156.5)
- moved J2 242.9 mm to (152.4, 144.3), turned to 180 degrees

Commit message: milestone 1
Parts:
- moved J2 210.1 mm to (183.1, -63.6)
- moved U1 208.1 mm to (141.5, -136.5)
- moved U13 208.1 mm to (141.5, -89.5)
- moved U22 208.1 mm to (139.6, -60.3)
- moved J3 208.1 mm to (121.8, -114.3)
- moved J4 208.1 mm to (187.2, -80.0)
- moved U10 208.1 mm to (102.1, -136.5)
- moved U11 208.1 mm to (69.1, -149.2)
- moved U12 208.1 mm to (83.1, -71.8)
- moved U14 208.1 mm to (153.5, -71.8)
- moved U15 208.1 mm to (102.1, -89.5)
- moved U16 208.1 mm to (65.3, -76.8)
- moved U19 208.1 mm to (151.6, -170.8)
- moved U2 208.1 mm to (159.9, -153.0)
- moved U20 208.1 mm to (177.0, -158.8)
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Routing:
- net GND: track 0.00 -> 631.3 mm
- net 3.3vUlSo: track 0.00 -> 411.9 mm
- net SDA: track 0.00 -> 403.8 mm
- net SCL: track 0.00 -> 402.3 mm
- net 5v: track 0.00 -> 235.1 mm
- net 3.3vDriverNode: track 0.00 -> 157.5 mm
- net 3.3vDACNode: track 0.00 -> 141.2 mm
- net CANH: track 0.00 -> 126.9 mm
- net CANL: track 0.00 -> 119.1 mm
- net 3.3vGPSNode: track 0.00 -> 75.8 mm
- net oledSCL: track 0.00 -> 68.1 mm, vias 0 -> 1
- net oledSDA: track 0.00 -> 65.5 mm, vias 0 -> 1
- net compSCL: track 0.00 -> 65.2 mm
- net outEnc: track 0.00 -> 63.6 mm
- net compSCA: track 0.00 -> 62.6 mm
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Other:
- net class Default: clearance 0.2 -> 0.3
- rule trace_clearance: 0.2 -> 0.3

Commit message: Commit Made on - April 29th 2021 @ :33:39
Routing:
- net GND: track 631.3 -> 654.1 mm
- net gpsRxGpsNode: track 55.3 -> 59.4 mm
- net SDA: track 403.8 -> 407.2 mm, vias 0 -> 1
- net 3.3vUlSo: track 411.9 -> 413.8 mm
- net Net-(J2-Pad1): track 33.9 -> 35.1 mm
- added copper zone on B.Cu, net GND
- added copper zone on F.Cu, net GND
