File: pcbDesignForAutonomousDrivingProject.kicad_pcb (KiCad board)
At the start: 2 copper layers, 145 x 145 mm, 24 parts, among them J1 Wheel Encoder, J2 Jack-DC, J3 CanHL, J4 Input, U1 can, U10 can, U11 GPSModule, U12 SJ2Board, U13 can, U14 SJ2Board, U15 can, U16 DAC, U17 motorTransceiver, U19 OLED, U2 SJ2Board, U20 ESP8266, U22 12vto5v, U3 SJ2Board, U4 Compass, U5 ultrasonic, U6 ultrasonic, U7 ultrasonic, U8 ultrasonic, U9 ultrasonic

Commit message: Commit Made on - April 29th 2021 @ 10:42:38 AM
Routing:
- net canRxcomp: track 34.1 -> 37.4 mm
- net GND: track 654.1 -> 656.9 mm
- net SDA: track 407.2 -> 409.7 mm
- net 3.3vDriverNode: track 157.5 -> 159.5 mm
- net CANH: track 126.9 -> 128.6 mm
- net 3.3vGPSNode: track 75.8 -> 77.4 mm
- net 3.3vDACNode: track 141.2 -> 142.4 mm
- net Net-(J2-Pad2): track 39.1 -> 40.2 mm
- net 3.3vbridgeNode: track 6.40 -> 7.54 mm
- net CANL: track 119.1 -> 119.9 mm
- net wifiTx: track 61.1 -> 61.9 mm
- net Net-(J2-Pad1): track 35.1 -> 35.9 mm
- net SCL: track 402.6 -> 403.3 mm
- net 3.3vUlSo: track 413.8 -> 414.5 mm
- net gpsTxGpsNode: track 52.1 -> 52.6 mm
Other:
- rule trace_min: 0.2 -> 0.4

Commit message: Commit Made on - April 29th 2021 @ 12:56:31 PM
Parts:
- added G***: LOGO, myFootprint:logo, F.Cu at (95.2, -160.0)
- moved U14 2.01 mm to (155.4, -71.1), turned to 180 degrees
- moved U3 1.57 mm to (87.9, -153.4), turned to 0 degrees
- moved U12 1.37 mm to (84.3, -71.1), turned to 180 degrees
- moved U2 0.97 mm to (159.0, -153.4), turned to 0 degrees
Routing:
- net 3.3vDriverNode: track 159.5 -> 101.1 mm, vias 0 -> 2
- net gpsRxGpsNode: track 59.4 -> 14.2 mm
- net 3.3vDACNode: track 142.4 -> 101.8 mm
- net GND: track 656.9 -> 620.5 mm
- net gpsTxGpsNode: track 52.6 -> 17.6 mm
- net SCLdac: track 29.3 -> 58.4 mm
- net SDAdac: track 29.3 -> 57.7 mm
- net outEnc: track 63.6 -> 91.4 mm
- net 3.3vUlSo: track 414.5 -> 436.6 mm
- net SDA: track 409.7 -> 425.0 mm, vias 1 -> 2
- net canRxcomp: track 37.4 -> 22.4 mm
- net canRX: track 35.2 -> 22.0 mm
- net canTxcomp: track 29.6 -> 16.7 mm
- net canTxGpsNode: track 24.3 -> 37.1 mm
- net canRxGpsNode: track 24.3 -> 37.1 mm
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