File: pcbDesignForAutonomousDrivingProject.sch (KiCad schematic (older format))
At the start: 3 parts

Commit message: Commit Made on - April 17th 2021 @ 01:57:31 PM
Parts:
- removed J?: ExternalDAC, symbol myComponents:ExternalDAC
- removed J?: Conn_01x04, symbol Connector_Generic:Conn_01x04
- added U? (x5): ultrasonic, symbol myComponents:ultrasonic
- added U?: can, symbol myComponents:can
Connections:
- net labels added: 3.3v, 5v, GND, SCL, SDA, canRX, canTx
- no-connect marks 0 -> 35
Other:
- moved on the sheet: U?
Changed lines of the file:
@@
 L myComponents:SJ2Board U?
 U 1 1 607A89AA
-P 2200 2300
-F 0 "U?" H 2200 3465 50  0000 C CNN
-F 1 "SJ2Board" H 2200 3374 50  0000 C CNN
-F 2 "" H 2200 1300 50  0001 C CNN
-F 3 "" H 2200 1300 50  0001 C CNN
-	1    2200 2300
+P 2600 2100
+F 0 "U?" H 2600 3265 50  0000 C CNN
+F 1 "SJ2Board" H 2600 3174 50  0000 C CNN
+F 2 "" H 2600 1100 50  0001 C CNN
+F 3 "" H 2600 1100 50  0001 C CNN
+	1    2600 2100
 	1    0    0    -1
 $EndComp
 $Comp
-L myComponents:ExternalDAC J?
-U 1 1 607E8440
-P 2200 4100
-F 0 "J?" H 2588 4164 50  0000 L CNN
-F 1 "ExternalDAC" H 2588 4073 50  0000 L CNN
-F 2 "" V 2200 4200 50  0001 C CNN
-F 3 "~" V 2200 4200 50  0001 C CNN
-	1    2200 4100
-	1    0    0    -1
+L myComponents:ultrasonic U?
+U 1 1 607B7CAD
+P 3600 1200
+F 0 "U?" V 3628 1428 50  0000 L CNN
+F 1 "ultrasonic" V 3695 1428 20  0000 L CNN
+F 2 "" H 3100 900 50  0001 C CNN
+F 3 "" H 3100 900 50  0001 C CNN
+	1    3600 1200
+	0    1    1    0
 $EndComp
 $Comp
-L Connector_Generic:Conn_01x04 J?
-U 1 1 607E9889
-P 1300 3100
-F 0 "J?" H 1380 3092 50  0000 L CNN
-F 1 "Conn_01x04" H 1380 3001 50  0000 L CNN
-F 2 "" H 1300 3100 50  0001 C CNN
-F 3 "~" H 1300 3100 50  0001 C CNN
-	1    1300 3100
-	1    0    0    -1
+L myComponents:ultrasonic U?
+U 1 1 607B88FD
+P 4300 1200
+F 0 "U?" V 4328 1428 50  0000 L CNN
+F 1 "ultrasonic" V 4395 1428 20  0000 L CNN
+F 2 "" H 3800 900 50  0001 C CNN
+F 3 "" H 3800 900 50  0001 C CNN
+	1    4300 1200
+	0    1    1    0
 $EndComp
+$Comp
+L myComponents:ultrasonic U?
+U 1 1 607B8C42
+P 5000 1200
+F 0 "U?" V 5028 1428 50  0000 L CNN
+F 1 "ultrasonic" V 5095 1428 20  0000 L CNN
+F 2 "" H 4500 900 50  0001 C CNN
+F 3 "" H 4500 900 50  0001 C CNN
+	1    5000 1200
+	0    1    1    0
+$EndComp
+$Comp
+L myComponents:ultrasonic U?
+U 1 1 607B8E5B
+P 5700 1200
+F 0 "U?" V 5728 1428 50  0000 L CNN
+F 1 "ultrasonic" V 5795 1428 20  0000 L CNN
+F 2 "" H 5200 900 50  0001 C CNN
+F 3 "" H 5200 900 50  0001 C CNN
+	1    5700 1200
+	0    1    1    0
+$EndComp
+$Comp
+L myComponents:ultrasonic U?
+U 1 1 607B9182
+P 6300 1200
+F 0 "U?" V 6328 1428 50  0000 L CNN
+F 1 "ultrasonic" V 6395 1428 20  0000 L CNN
+F 2 "" H 5800 900 50  0001 C CNN
+F 3 "" H 5800 900 50  0001 C CNN
+	1    6300 1200
+	0    1    1    0
+$EndComp
+Text GLabel 3500 1300 0    39   Input ~ 0
+SCL
+Text GLabel 4200 1300 0    39   Input ~ 0
+SCL
+Text GLabel 4900 1300 0    39   Input ~ 0
+SCL
+Text GLabel 5600 1300 0    39   Input ~ 0
+SCL
+Text GLabel 3500 1400 0    39   Input ~ 0
+SDA
+Text GLabel 4200 1400 0    39   Input ~ 0
+SDA
+Text GLabel 4900 1400 0    39   Input ~ 0
+SDA
+Text GLabel 5600 1400 0    39   Input ~ 0
+SDA
+Text GLabel 3100 3000 2    39   Input ~ 0
+SCL
+Text GLabel 6200 1300 0    39   Input ~ 0
+SCL
+Text GLabel 6200 1400 0    39   Input ~ 0
+SDA
+Text GLabel 2100 3000 0    39   Input ~ 0
+SDA
+Text GLabel 3500 1100 0    39   Input ~ 0
+3.3v
+Text GLabel 4200 1100 0    39   Input ~ 0
+3.3v
+Text GLabel 4900 1100 0    39   Input ~ 0
+3.3v
+Text GLabel 5600 1100 0    39   Input ~ 0
+3.3v
+Text GLabel 6200 1100 0    39   Input ~ 0
+3.3v
+Text GLabel 3500 1200 0    39   Input ~ 0
+GND
+Text GLabel 4200 1200 0    39   Input ~ 0
+GND
+Text GLabel 4900 1200 0    39   Input ~ 0
+GND
+Text GLabel 5600 1200 0    39   Input ~ 0
+GND
+Text GLabel 6200 1200 0    39   Input ~ 0
+GND
+Text GLabel 3100 1200 2    39   Input ~ 0
+5v
+NoConn ~ 3100 1300
+NoConn ~ 3100 1400
+NoConn ~ 3100 1500
+NoConn ~ 3100 1600
+NoConn ~ 3100 1700
+NoConn ~ 3100 1800
+NoConn ~ 3100 1900
+NoConn ~ 3100 2000
+NoConn ~ 3100 2500
+NoConn ~ 3100 2400
+NoConn ~ 3100 2600
+NoConn ~ 3100 2800
+NoConn ~ 3100 2700
+NoConn ~ 3100 2900
+NoConn ~ 3100 2100
+NoConn ~ 3100 2200
+NoConn ~ 3100 2300
+NoConn ~ 2100 2900
+NoConn ~ 2100 2800
+NoConn ~ 2100 2700
+NoConn ~ 2100 2600
+NoConn ~ 2100 2500
+NoConn ~ 2100 2400
+NoConn ~ 2100 2300
+NoConn ~ 2100 2200
+NoConn ~ 2100 2100
+NoConn ~ 2100 2000
+NoConn ~ 2100 1900
+NoConn ~ 2100 1800
+NoConn ~ 2100 1700
+NoConn ~ 2100 1600
+NoConn ~ 2100 1200
+NoConn ~ 2100 1300
+NoConn ~ 2100 1400
+NoConn ~ 2100 1500
+Text GLabel 3100 3100 2    39   Input ~ 0
+GND
+Text GLabel 2100 3100 0    39   Input ~ 0
+GND
+Wire Notes Line
+	500  600  6900 600
+Wire Notes Line
+	6900 600  6900 1900
+Wire Notes Line
+	6900 1900 3700 1900
+Wire Notes Line
+	3700 1900 3700 3500
+Wire Notes Line
+	3700 3500 500  3500
+Wire Notes Line
+	500  3500 500  600
+Text GLabel 1700 1400 2    39   Input ~ 0
+GND
+Text GLabel 1700 1300 2    39   Input ~ 0
+3.3v
+Text GLabel 1700 1500 2    39   Input ~ 0
+canRX
+$Comp
+L myComponents:can U?
+U 1 1 607BC269
+P 1100 1400
+F 0 "U?" V 1465 1300 50  0000 C CNN
+F 1 "can" V 1374 1300 50  0000 C CNN
+F 2 "" H 600 2100 50  0001 C CNN
+F 3 "" H 600 2100 50  0001 C CNN
+	1    1100 1400
+	0    -1   -1   0
+$EndComp
+Text GLabel 1700 1600 2    39   Input ~ 0
+canTx
 $EndSCHEMATC

Commit message: Commit Made on - April 18th 2021 @ 04:05:23 PM
Parts:
- added C?: C, symbol Device:R
- added J?: Wheel Encoder, symbol myComponents:Encoder
- added R?: R, symbol Device:R
- added U?: SJ2Board, symbol myComponents:SJ2Board
Connections:
- net labels added: VCC, outEnc
- wire segments 0 -> 8
- no-connect marks 35 -> 36
Other:
- moved on the sheet: U?

Commit message: Commit Made on - April 22th 2021 @ :52:41
Parts:
- added U10, U13, U15, U18: can, symbol myComponents:can
- added U11: GPSModule, symbol myComponents:GPSModule
- added U14, U21, U3: SJ2Board, symbol myComponents:SJ2Board
- added U16: DAC, symbol myComponents:DAC
- added U17: motorTransceiver, symbol myComponents:motorTransceiver
- added U19: OLED, symbol myComponents:OLED
- added U20: ESP8266, symbol myComponents:ESP8266
- added U4: Compass, symbol myComponents:Compass
- gave numbers to parts that had none: 11
Connections:
- net labels added: CANH, CANL, SCLdac, SDAdac, canRxBrNd, canRxDrNd, canRxGpsNode, canRxcomp, canTX, canTxBrNd, canTxDrNd, canTxGpsNode, canTxcomp, com3, compSCA, compSCL, gpsRxGpsNode, gpsTxGpsNode, oledSCL, oledSDA, wifiRx, wifiTx
- net labels removed: VCC, canTx
- wire segments 8 -> 22
- no-connect marks 36 -> 174
Other:
- note added: "Bridge Node"
- note added: "Driver Node"
- note added: "GPS Node"
- note added: "Ultrasonic"
- note added: "motorTransceiver Dac"
- moved on the sheet: U1

Commit message: Commit Made on - April 22th 2021 @ 11:12:07 AM
Parts:
- C1: footprint (none) -> Capacitor_THT:CP_Radial_D8.0mm_P3.80mm
- R1: footprint (none) -> Resistor_THT:R_Axial_DIN0309_L9.0mm_D3.2mm_P2.54mm_Vertical
- U12, U14, U2, U21, U3: footprint (none) -> myFootprint:sj2Board
- U5, U6, U7, U8, U9: footprint (none) -> myFootprint:ultrasonic
Connections:
- no-connect marks 174 -> 173
Changed lines of the file:
@@
 F 0 "U2" H 1300 4065 50  0000 C CNN
 F 1 "SJ2Board" H 1300 3974 50  0000 C CNN
-F 2 "" H 1300 1900 50  0001 C CNN
+F 2 "myFootprint:sj2Board" H 1300 1900 50  0001 C CNN
 F 3 "" H 1300 1900 50  0001 C CNN
 	1    1300 2900
@@
 F 0 "U5" V 2528 1228 50  0000 L CNN
 F 1 "ultrasonic" V 2595 1228 20  0000 L CNN
-F 2 "" H 2000 700 50  0001 C CNN
+F 2 "myFootprint:ultrasonic" H 2000 700 50  0001 C CNN
 F 3 "" H 2000 700 50  0001 C CNN
 	1    2500 1000
@@
 F 0 "U7" V 2528 2628 50  0000 L CNN
 F 1 "ultrasonic" V 2595 2628 20  0000 L CNN
-F 2 "" H 2000 2100 50  0001 C CNN
+F 2 "myFootprint:ultrasonic" H 2000 2100 50  0001 C CNN
 F 3 "" H 2000 2100 50  0001 C CNN
 	1    2500 2400
@@
 F 0 "U6" V 2528 1928 50  0000 L CNN
 F 1 "ultrasonic" V 2595 1928 20  0000 L CNN
-F 2 "" H 2000 1400 50  0001 C CNN
+F 2 "myFootprint:ultrasonic" H 2000 1400 50  0001 C CNN
 F 3 "" H 2000 1400 50  0001 C CNN
 	1    2500 1700
@@
 F 0 "U8" V 2528 3328 50  0000 L CNN
 F 1 "ultrasonic" V 2595 3328 20  0000 L CNN
-F 2 "" H 2000 2800 50  0001 C CNN
+F 2 "myFootprint:ultrasonic" H 2000 2800 50  0001 C CNN
 F 3 "" H 2000 2800 50  0001 C CNN
 	1    2500 3100
@@
 F 0 "U9" V 2528 4028 50  0000 L CNN
 F 1 "ultrasonic" V 2595 4028 20  0000 L CNN
-F 2 "" H 2000 3500 50  0001 C CNN
+F 2 "myFootprint:ultrasonic" H 2000 3500 50  0001 C CNN
 F 3 "" H 2000 3500 50  0001 C CNN
 	1    2500 3800
@@
 F 0 "U12" H 4150 4165 50  0000 C CNN
 F 1 "SJ2Board" H 4150 4074 50  0000 C CNN
-F 2 "" H 4150 2000 50  0001 C CNN
+F 2 "myFootprint:sj2Board" H 4150 2000 50  0001 C CNN
 F 3 "" H 4150 2000 50  0001 C CNN
 	1    4150 3000
@@
 Wire Notes Line
 	600  700  3100 700
-$Comp
-L myComponents:Encoder J1
-U 1 1 607F3B01
-P 4300 1000
-F 0 "J1" H 4478 1092 50  0000 L CNN
-F 1 "Wheel Encoder" H 4100 800 50  0000 L CNN
-F 2 "" H 4200 1100 50  0001 C CNN
-F 3 "~" H 4200 1100 50  0001 C CNN
-	1    4300 1000
-	1    0    0    -1
-$EndComp
 Text GLabel 4000 800  0    50   Input ~ 0
 3.3v
 Text GLabel 4000 900  0    50   Input ~ 0
 GND
-NoConn ~ 4000 1000
 $Comp
 L Device:R R1
@@
 F 0 "R1" V 4200 1500 50  0000 C CNN
 F 1 "R" V 4300 1500 50  0000 C CNN
-F 2 "" V 4230 1500 50  0001 C CNN
+F 2 "Resistor_THT:R_Axial_DIN0309_L9.0mm_D3.2mm_P2.54mm_Vertical" V 4230 1500 50  0001 C CNN
 F 3 "~" H 4300 1500 50  0001 C CNN
 	1    4300 1500
@@
 F 0 "C1" V 3700 1500 50  0000 C CNN
 F 1 "C" V 3800 1500 50  0000 C CNN
-F 2 "" V 3730 1500 50  0001 C CNN
+F 2 "Capacitor_THT:CP_Radial_D8.0mm_P3.80mm" V 3730 1500 50  0001 C CNN
 F 3 "~" H 3800 1500 50  0001 C CNN
 	1    3800 1500
@@
 Wire Wire Line
 	4550 1300 3900 1300
-Wire Wire Line
-	3900 1300 3900 1100
-Wire Wire Line
-	3900 1100 4000 1100
 Wire Wire Line
 	4150 1500 4050 1500
@@
 F 0 "U3" H 1550 6915 50  0000 C CNN
 F 1 "SJ2Board" H 1550 6824 50  0000 C CNN
-F 2 "" H 1550 4750 50  0001 C CNN
+F 2 "myFootprint:sj2Board" H 1550 4750 50  0001 C CNN
 F 3 "" H 1550 4750 50  0001 C CNN
 	1    1550 5750
@@
 F 0 "U14" H 5550 6815 50  0000 C CNN
 F 1 "SJ2Board" H 5550 6724 50  0000 C CNN
-F 2 "" H 5550 4650 50  0001 C CNN
+F 2 "myFootprint:sj2Board" H 5550 4650 50  0001 C CNN
 F 3 "" H 5550 4650 50  0001 C CNN
 	1    5550 5650
@@
 F 0 "U21" H 10050 6015 50  0000 C CNN
 F 1 "SJ2Board" H 10050 5924 50  0000 C CNN
-F 2 "" H 10050 3850 50  0001 C CNN
+F 2 "myFootprint:sj2Board" H 10050 3850 50  0001 C CNN
 F 3 "" H 10050 3850 50  0001 C CNN
 	1    10050 4850
@@
 Text GLabel 8050 6200 2    39   Input ~ 0
 5v
+$Comp
+L myComponents:Encoder J1
+U 1 1 607F3B01
+P 4300 1000
+F 0 "J1" H 4478 1092 50  0000 L CNN
+F 1 "Wheel Encoder" H 4100 800 50  0000 L CNN
+F 2 "" H 4200 1100 50  0001 C CNN
+F 3 "~" H 4200 1100 50  0001 C CNN
+	1    4300 1000
+	1    0    0    -1
+$EndComp
+Wire Wire Line
+	4000 1000 3900 1000
+Wire Wire Line
+	3900 1000 3900 1300
 $EndSCHEMATC

Commit message: Commit Made on - April 22th 2021 @ 03:50:36 PM
Parts:
- U11: footprint (none) -> myFootprint:GPS
- U16: footprint (none) -> myFootprint:DAC
- U17: footprint (none) -> myFootprint:motorTransceiver
- U19: footprint (none) -> myFootprint:Oled
- U20: footprint (none) -> myFootprint:ESP8266
- U4: footprint (none) -> myFootprint:compass
Changed lines of the file:
@@
 F 0 "U11" H 2650 5050 50  0000 L CNN
 F 1 "GPSModule" H 3000 4900 50  0000 L CNN
-F 2 "" H 3150 4800 50  0001 C CNN
+F 2 "myFootprint:GPS" H 3150 4800 50  0001 C CNN
 F 3 "" H 3150 4800 50  0001 C CNN
 	1    3150 4800
@@
 F 0 "U4" H 1150 7300 50  0000 L CNN
 F 1 "Compass" H 1350 7250 50  0000 L CNN
-F 2 "" H 900 6550 50  0001 C CNN
+F 2 "myFootprint:compass" H 900 6550 50  0001 C CNN
 F 3 "" H 900 6550 50  0001 C CNN
 	1    1600 7150
@@
 F 0 "U20" H 7850 5050 50  0000 C CNN
 F 1 "ESP8266" V 7850 5250 39  0000 C CNN
-F 2 "" H 7850 5300 50  0001 C CNN
+F 2 "myFootprint:ESP8266" H 7850 5300 50  0001 C CNN
 F 3 "" H 7850 5300 50  0001 C CNN
 	1    7850 5300
@@
 F 0 "U19" V 7750 6450 50  0000 C CNN
 F 1 "OLED" V 7900 6450 50  0000 C CNN
-F 2 "" H 7550 5700 50  0001 C CNN
+F 2 "myFootprint:Oled" H 7550 5700 50  0001 C CNN
 F 3 "" H 7550 5700 50  0001 C CNN
 	1    7750 6100
@@
 F 0 "U17" H 6578 2118 79  0000 L CNN
 F 1 "motorTransceiver" H 5850 1700 79  0000 L CNN
-F 2 "" H 5750 1600 79  0001 C CNN
+F 2 "myFootprint:motorTransceiver" H 5750 1600 79  0001 C CNN
 F 3 "" H 5750 1600 79  0001 C CNN
 	1    6350 2100
@@
 F 0 "U16" H 6478 3318 79  0000 L CNN
 F 1 "DAC" H 6478 3183 79  0000 L CNN
-F 2 "" H 5850 2900 79  0001 C CNN
+F 2 "myFootprint:DAC" H 5850 2900 79  0001 C CNN
 F 3 "" H 5850 2900 79  0001 C CNN
 	1    6250 3200

Commit message: Commit Made on - April 22th 2021 @ 08:30:16 PM
Parts:
- J1: footprint (none) -> myFootprint:WheelEncoder
- U1, U10, U13, U15, U18: footprint (none) -> myFootprint:can
Changed lines of the file:
@@
 F 0 "U1" V 1000 1450 50  0000 C CNN
 F 1 "can" V 1400 1100 50  0000 C CNN
-F 2 "" H 750 1900 50  0001 C CNN
+F 2 "myFootprint:can" H 750 1900 50  0001 C CNN
 F 3 "" H 750 1900 50  0001 C CNN
 	1    1250 1200
@@
 F 0 "U10" V 3415 6000 50  0000 C CNN
 F 1 "can" V 3324 6000 50  0000 C CNN
-F 2 "" H 2550 6800 50  0001 C CNN
+F 2 "myFootprint:can" H 2550 6800 50  0001 C CNN
 F 3 "" H 2550 6800 50  0001 C CNN
 	1    3050 6100
@@
 F 0 "U13" V 5665 7150 50  0000 C CNN
 F 1 "can" V 5574 7150 50  0000 C CNN
-F 2 "" H 4800 7950 50  0001 C CNN
+F 2 "myFootprint:can" H 4800 7950 50  0001 C CNN
 F 3 "" H 4800 7950 50  0001 C CNN
 	1    5300 7250
@@
 F 0 "U18" V 7600 4650 50  0000 C CNN
 F 1 "can" V 7850 4600 50  0000 C CNN
-F 2 "" H 7250 5400 50  0001 C CNN
+F 2 "myFootprint:can" H 7250 5400 50  0001 C CNN
 F 3 "" H 7250 5400 50  0001 C CNN
 	1    7750 4700
@@
 F 0 "U15" V 5550 1350 50  0000 C CNN
 F 1 "can" V 5950 1000 50  0000 C CNN
-F 2 "" H 5300 1800 50  0001 C CNN
+F 2 "myFootprint:can" H 5300 1800 50  0001 C CNN
 F 3 "" H 5300 1800 50  0001 C CNN
 	1    5800 1100
@@
 F 0 "J1" H 4478 1092 50  0000 L CNN
 F 1 "Wheel Encoder" H 4100 800 50  0000 L CNN
-F 2 "" H 4200 1100 50  0001 C CNN
+F 2 "myFootprint:WheelEncoder" H 4200 1100 50  0001 C CNN
 F 3 "~" H 4200 1100 50  0001 C CNN
 	1    4300 1000

Commit message: Commit Made on - April 23th 2021 @ 08:27:51 PM
Parts:
- added J2: Jack-DC, Connector_BarrelJack:BarrelJack_CUI_PJ-102AH_Horizontal, symbol Connector:Jack-DC
- added U22: 12vto5v, myFootprint:12vto5v, symbol myComponents:12vto5v
Connections:
- net 5v: now also U22.3 (5v+)
- net GND: now also U22.4 (5v-)
- new net: J2.1, U22.1 (12v+)
- new net: J2.2, U22.2 (12v-)
Other:
- note added: "Mains 12v to 5v"
Changed lines of the file:
@@
 Wire Wire Line
 	3900 1000 3900 1300
+$Comp
+L myComponents:12vto5v U22
+U 1 1 6083A09C
+P 10300 2200
+F 0 "U22" H 10300 2549 50  0000 C CNN
+F 1 "12vto5v" H 10300 2466 39  0000 C CNN
+F 2 "myFootprint:12vto5v" H 9700 1600 50  0001 C CNN
+F 3 "" H 9700 1600 50  0001 C CNN
+	1    10300 2200
+	1    0    0    -1
+$EndComp
+Wire Notes Line
+	11150 3550 8450 3550
+Wire Notes Line
+	8450 3550 8450 700
+Wire Notes Line
+	8450 700  11150 700
+Wire Notes Line
+	11150 700  11150 3550
+Text Notes 9150 1100 0    118  ~ 24
+Mains 12v to 5v
+Text GLabel 10700 2300 2    39   Input ~ 0
+GND
+Text GLabel 10700 2100 2    39   Input ~ 0
+5v
+$Comp
+L Connector:Jack-DC J2
+U 1 1 60841F9D
+P 9050 2200
+F 0 "J2" H 9107 2525 50  0000 C CNN
+F 1 "Jack-DC" H 9107 2434 50  0000 C CNN
+F 2 "Connector_BarrelJack:BarrelJack_CUI_PJ-102AH_Horizontal" H 9100 2160 50  0001 C CNN
+F 3 "~" H 9100 2160 50  0001 C CNN
+	1    9050 2200
+	1    0    0    -1
+$EndComp
+Wire Wire Line
+	9900 2100 9350 2100
+Wire Wire Line
+	9350 2300 9900 2300
 $EndSCHEMATC

Commit message: Commit Made on - April 25th 2021 @ 11:22:35 PM
Parts:
- added J3: CanHL, Connector_PinHeader_2.54mm:PinHeader_1x02_P2.54mm_Vertical, symbol Connector_Generic:Conn_01x02
- C1: footprint Capacitor_THT:CP_Radial_D8.0mm_P3.80mm -> Capacitor_THT:CP_Radial_D5.0mm_P2.50mm
Connections:
- net 5v: no longer U17.1 (Vdd)
- net CANH: now also J3.2 (Pin_2)
- net CANL: now also J3.1 (Pin_1)
- net 3.3vUlSo: now reaches U2.4 (Vcc-3.3v)
- net 3.3vUlSo: now also U1.3 (3.3), U5.1 (Vcc), U6.1 (Vcc), U7.1 (Vcc), U8.1 (Vcc), U9.1 (Vcc)
- net 3.3vDACNode: now reaches U12.4 (Vcc-3.3v)
- net 3.3vDACNode: now also J1.1 (VCC), U15.3 (3.3), U17.1 (Vdd)
- net 3.3vGPSNode: now reaches U3.4 (Vcc-3.3v)
- net 3.3vGPSNode: now also U10.3 (3.3), U11.0 (3.3v), U4.7 (3.3v)
- net 3.3vDriverNode: now reaches U14.4 (Vcc-3.3v)
- net 3.3vDriverNode: now also U13.3 (3.3)
- net 3.3vbridgeNode: now reaches U21.4 (Vcc-3.3v)
- net 3.3vbridgeNode: now also U18.3 (3.3), U20.5 (EN), U20.7 (3.3v)
- removed net 3.3v: J1.1 (VCC), U1.3 (3.3), U10.3 (3.3), U11.0 (3.3v), U13.3 (3.3), U15.3 (3.3), U18.3 (3.3), U20.5 (EN), U20.7 (3.3v), U4.7 (3.3v), U5.1 (Vcc), U6.1 (Vcc), U7.1 (Vcc), U8.1 (Vcc), U9.1 (Vcc)
- no-connect marks 173 -> 168
Other:
- note added: "Ultrasonic Node"
- note added: "motorTxRx Node"
- note removed: "Ultrasonic"
- note removed: "motorTransceiver Dac"
