File: pcbDesignForAutonomousDrivingProject.sch (KiCad schematic (older format))
At the start: 27 parts, among them J1 Wheel Encoder, J2 Jack-DC, J3 CanHL, U1 can, U10 can, U11 GPSModule, U12 SJ2Board, U13 can, U14 SJ2Board, U15 can, U16 DAC, U17 motorTransceiver, U18 can, U19 OLED, U2 SJ2Board, U20 ESP8266, U21 SJ2Board, U22 12vto5v, U3 SJ2Board, U4 Compass, U5 ultrasonic, U6 ultrasonic, U7 ultrasonic, U8 ultrasonic, U9 ultrasonic

Commit message: Commit Made on - April 28th 2021 @ 11:39:06 PM
Parts:
- removed C1: C, Capacitor_THT:CP_Radial_D5.0mm_P2.50mm, symbol Device:R
- removed R1: R, Resistor_THT:R_Axial_DIN0309_L9.0mm_D3.2mm_P2.54mm_Vertical, symbol Device:R
- removed U18: can, myFootprint:can, symbol myComponents:can
- removed U21: SJ2Board, myFootprint:sj2Board, symbol myComponents:SJ2Board
- J2: footprint Connector_BarrelJack:BarrelJack_CUI_PJ-102AH_Horizontal -> myFootprint:BarrelJack_Horizontal
Connections:
- net 3.3vDACNode: now also U16.1 (VDD); no longer J1.1 (VCC)
- net 3.3vDriverNode: now also U19.1 (GND)
- net 5v: now also J1.1 (VCC); no longer U16.1 (VDD), U19.0 (VCC)
- net GND: now also U19.0 (VCC); no longer U19.1 (GND)
- net oledSCL: now also U14.15 (P1.31)
- net oledSDA: now also U14.16 (P1.30)
- net outEnc: now also J1.3 (D0)
- net wifiRx: now also U2.31 (P0.15)
- net wifiTx: now also U2.30 (P0.16)
- no-connect marks 168 -> 134
Other:
- note removed: "Bridge Node"
- moved on the sheet: J1, U12, U15, U16, U17, U19, U20

Commit message: Commit Made on - April 29th 2021 @ :36:51
Parts:
- added J?: Input, Connector_PinHeader_2.54mm:PinHeader_1x02_P2.54mm_Vertical, symbol Connector_Generic:Conn_01x02
Connections:
- net at J2.1, U22.1 (12v+): now also J?.1 (Pin_1)
- net at J2.2, U22.2 (12v-): now also J?.2 (Pin_2)
Changed lines of the file:
@@
 $EndComp
-Wire Wire Line
-	9900 2100 9350 2100
 Wire Wire Line
 	9350 2300 9900 2300
@@
 Text GLabel 7600 5600 2    39   Input ~ 0
 GND
-Text GLabel 7600 5500 2    39   Input ~ 0
-3.3vDriverNode
 Text GLabel 1800 2100 2    39   Input ~ 0
 3.3vUlSo
@@
 Text GLabel 7600 5300 2    39   Input ~ 0
 oledSDA
+Wire Wire Line
+	9900 2100 9350 2100
+Text GLabel 7600 5500 2    39   Input ~ 0
+3.3vDriverNode
+$Comp
+L Connector_Generic:Conn_01x02 J?
+U 1 1 60946026
+P 9650 1650
+F 0 "J?" H 9730 1642 50  0000 L CNN
+F 1 "Input" H 9730 1551 50  0000 L CNN
+F 2 "Connector_PinHeader_2.54mm:PinHeader_1x02_P2.54mm_Vertical" H 9650 1650 50  0001 C CNN
+F 3 "~" H 9650 1650 50  0001 C CNN
+	1    9650 1650
+	0    1    1    0
+$EndComp
+Wire Wire Line
+	9900 2100 9900 1450
+Wire Wire Line
+	9900 1450 9650 1450
+Connection ~ 9900 2100
+Wire Wire Line
+	9550 1450 8750 1450
+Wire Wire Line
+	8750 1450 8750 2550
+Wire Wire Line
+	8750 2550 9900 2550
+Wire Wire Line
+	9900 2550 9900 2300
+Connection ~ 9900 2300
 $EndSCHEMATC

Commit message: Commit Made on - April 29th 2021 @ :52:21
Parts:
- gave numbers to parts that had none: 1
Changed lines of the file:
@@
 3.3vDriverNode
 $Comp
-L Connector_Generic:Conn_01x02 J?
+L Connector_Generic:Conn_01x02 J4
 U 1 1 60946026
 P 9650 1650
-F 0 "J?" H 9730 1642 50  0000 L CNN
+F 0 "J4" H 9730 1642 50  0000 L CNN
 F 1 "Input" H 9730 1551 50  0000 L CNN
 F 2 "Connector_PinHeader_2.54mm:PinHeader_1x02_P2.54mm_Vertical" H 9650 1650 50  0001 C CNN
